File: board/unijoysticle/_saved_unijoysticle.sch (KiCad schematic (older format))
At the start: 9 parts, among them J1 DB9_Female_MountingHoles, J2 DB9_Female_MountingHoles, J3 Barrel_Jack_MountingPin, U1 4066, U2 4066, U4 4066, U5 4066

Commit message: board: MH-ET live kind of Okish...
Parts:
- B1: footprint RF_Module:ESP32-WROOM-32 -> Parts:MH-ET_LIVE_MINIKIT_ESP32
Changed lines of the file:
@@
 F 0 "B1" H 5250 5560 45  0000 C CNN
 F 1 "ESP32_THING_W_ANT_KEEPOUT" H 5250 5476 45  0000 C CNN
-F 2 "RF_Module:ESP32-WROOM-32" H 5250 5400 20  0001 C CNN
+F 2 "Parts:MH-ET_LIVE_MINIKIT_ESP32" H 5250 5400 20  0001 C CNN
 F 3 "" H 5250 4200 50  0001 C CNN
 F 4 "DEV-13907" H 5250 5381 60  0000 C CNN "Field4"
