File: board/unijoysticle2plus/unijoysticle2plus.sch (KiCad schematic (older format))
At the start: 45 parts, among them J1 DB9_Female, J2 DB9_Female, J3 USB_B_Micro, Q1 S8050, Q2 S8050, SW1 RESET, SW2 JOY SWAP, U1 74HC05, U2 74HC05, U3 74HC05, U4 ESP32-WROOM-32D, U5 AMS1117-3.3, U6 CP2102N-A01-GQFN28

Commit message: unijoysticle2plus: REV A finished
- Includes footprint for USB Micro B
- Uses different ESD USB component, one that is available in JLCPCB
- Layout of CP2102 + ESD is a bit different
Parts:
- D6: LCSC C7074 -> C720028
- J3: footprint Connector_USB:USB_Micro-B_Molex-105017-0001 -> Connector_USB:USB_Micro-B_Molex_47346-0001; LCSC (none) -> C132560
- U6: value CP2102N-A01-GQFN28 -> CP2102
Other:
- note added: "Only 2102.\nRequires additional resistors for cp2102N"
- note removed: "Either a cp2102 or cp2102N"
Changed lines of the file:
@@
 F 0 "J3" H 7507 3017 50  0000 C CNN
 F 1 "USB_B_Micro" H 7507 2926 50  0000 C CNN
-F 2 "Connector_USB:USB_Micro-B_Molex-105017-0001" H 7600 2500 50  0001 C CNN
+F 2 "Connector_USB:USB_Micro-B_Molex_47346-0001" H 7600 2500 50  0001 C CNN
 F 3 "~" H 7600 2500 50  0001 C CNN
+F 4 "C132560" H 7450 2550 50  0001 C CNN "LCSC"
 	1    7450 2550
 	1    0    0    -1
@@
 USBD-
 Wire Wire Line
-	10050 5050 10050 5150
+	10050 5050 10050 5080
 $Comp
 L power:GND #PWR033
 U 1 1 60E6428D
-P 10050 5150
-F 0 "#PWR033" H 10050 4900 50  0001 C CNN
-F 1 "GND" H 10055 4977 50  0000 C CNN
-F 2 "" H 10050 5150 50  0001 C CNN
-F 3 "" H 10050 5150 50  0001 C CNN
-	1    10050 5150
+P 10050 5080
+F 0 "#PWR033" H 10050 4830 50  0001 C CNN
+F 1 "GND" H 10055 4907 50  0000 C CNN
+F 2 "" H 10050 5080 50  0001 C CNN
+F 3 "" H 10050 5080 50  0001 C CNN
+	1    10050 5080
 	1    0    0    -1
 $EndComp
@@
 P 10050 3750
 F 0 "U6" H 10250 2350 50  0000 C CNN
-F 1 "CP2102N-A01-GQFN28" H 10650 2450 50  0000 C CNN
+F 1 "CP2102" H 10270 2450 50  0000 C CNN
 F 2 "Package_DFN_QFN:QFN-28-1EP_5x5mm_P0.5mm_EP3.35x3.35mm" H 10500 2550 50  0001 L CNN
 F 3 "https://www.silabs.com/documents/public/data-sheets/cp2102n-datasheet.pdf" H 10100 3000 50  0001 C CNN
@@
 F 2 "Package_TO_SOT_SMD:SOT-143" H 8325 2850 50  0001 L CNN
 F 3 "http://www.littelfuse.com/~/media/files/littelfuse/technical%20resources/documents/data%20sheets/sp05xxba.pdf" H 8225 3025 50  0001 C CNN
-F 4 "C7074" H 8100 2900 50  0001 C CNN "LCSC"
+F 4 "C720028" H 8100 2900 50  0001 C CNN "LCSC"
 	1    8100 2900
 	1    0    0    -1
@@
 	0    -1   -1   0
 $EndComp
-Text Notes 10010 5430 0    50   ~ 0
-Either a cp2102 or cp2102N
 Text Notes 530  7700 0    50   ~ 0
 To prevent keyboard and/or other weird issues,\n7405 must be connected to C64 power lines (VDD)
@@
 	4100 1800 4100 1840
 Connection ~ 4100 1550
+Text Notes 9350 5380 0    50   ~ 0
+Only 2102.\nRequires additional resistors for cp2102N
 $EndSCHEMATC

Commit message: unijoysticle2plus: schematic cosmetic fixes
cosmetic fixes to make it more readable.
Other:
- note added: "Available GPIOs for future use.\nGPIOs 34-39 are Input only"
- moved on the sheet: H1, H2, H3, H4
Changed lines of the file:
@@
 	1    0    0    -1
 $EndComp
-Text Label 4300 1550 0    50   ~ 0
+Text Label 3550 1550 0    50   ~ 0
 ESP_EN
 $Comp
@@
 	1    0    0    -1
 $EndComp
-Text Label 6300 1550 2    50   ~ 0
+Text Label 6650 1550 2    50   ~ 0
 ESP_BOOT
 $Comp
@@
 GPIO_J2_POTY
 Wire Wire Line
-	5850 3750 6300 3750
-Wire Wire Line
-	5850 3850 6300 3850
-Text Label 6300 3750 2    50   ~ 0
+	5850 3750 6650 3750
+Wire Wire Line
+	5850 3850 6650 3850
+Text Label 6650 3750 2    50   ~ 0
 GPIO34
-Text Label 6300 3850 2    50   ~ 0
+Text Label 6650 3850 2    50   ~ 0
 GPIO35
 Wire Notes Line
@@
 U 1 1 5F96CB69
 P 6150 6000
-F 0 "D2" H 6000 6150 50  0000 C CNN
-F 1 "LED J1" H 6000 6050 50  0000 C CNN
+F 0 "D2" H 5900 6090 50  0000 C CNN
+F 1 "LED J1" H 6130 6090 50  0000 C CNN
 F 2 "LED_SMD:LED_0603_1608Metric_Pad1.05x0.95mm_HandSolder" H 6150 6000 50  0001 C CNN
 F 3 "~" H 6150 6000 50  0001 C CNN
@@
 U 1 1 5F96DEB5
 P 6150 6250
-F 0 "D3" H 6000 6400 50  0000 C CNN
-F 1 "LED J2" H 6000 6300 50  0000 C CNN
+F 0 "D3" H 5910 6340 50  0000 C CNN
+F 1 "LED J2" H 6140 6340 50  0000 C CNN
 F 2 "LED_SMD:LED_0603_1608Metric_Pad1.05x0.95mm_HandSolder" H 6150 6250 50  0001 C CNN
 F 3 "~" H 6150 6250 50  0001 C CNN
@@
 U 1 1 5F9908EC
 P 6550 6250
-F 0 "R4" V 6450 6250 50  0000 C CNN
-F 1 "150" V 6550 6250 50  0000 C CNN
+F 0 "R4" V 6470 6250 50  0000 C CNN
+F 1 "150" V 6630 6250 50  0000 C CNN
 F 2 "Resistor_SMD:R_0402_1005Metric" V 6480 6250 50  0001 C CNN
 F 3 "~" H 6550 6250 50  0001 C CNN
@@
 NoConn ~ 7750 2750
 Wire Wire Line
-	5850 1650 6300 1650
-Wire Wire Line
-	5850 1850 6300 1850
-Text Label 6300 1650 2    50   ~ 0
+	5850 1650 6650 1650
+Wire Wire Line
+	5850 1850 6650 1850
+Text Label 6650 1650 2    50   ~ 0
 ESP_TXD
-Text Label 6300 1850 2    50   ~ 0
+Text Label 6650 1850 2    50   ~ 0
 ESP_RXD
 Wire Wire Line
-	5850 1950 6300 1950
-Text Label 6300 1950 2    50   ~ 0
+	5850 1950 6650 1950
+Text Label 6650 1950 2    50   ~ 0
 GPIO04
 Wire Wire Line
@@
 U 1 1 60AF2CFC
 P 7900 4350
-F 0 "R5" V 7800 4350 50  0000 C CNN
-F 1 "10k" V 7900 4350 50  0000 C CNN
+F 0 "R5" V 7810 4350 50  0000 C CNN
+F 1 "10k" V 7980 4350 50  0000 C CNN
 F 2 "Resistor_SMD:R_0402_1005Metric" V 7830 4350 50  0001 C CNN
 F 3 "~" H 7900 4350 50  0001 C CNN
@@
 U 1 1 60AF3FED
 P 7900 4900
-F 0 "R6" V 8000 4900 50  0000 C CNN
-F 1 "10k" V 7900 4900 50  0000 C CNN
+F 0 "R6" V 7980 4900 50  0000 C CNN
+F 1 "10k" V 7800 4900 50  0000 C CNN
 F 2 "Resistor_SMD:R_0402_1005Metric" V 7830 4900 50  0001 C CNN
 F 3 "~" H 7900 4900 50  0001 C CNN
@@
 ESP_EN
 Wire Wire Line
-	5850 1550 6300 1550
+	5850 1550 6650 1550
 $Comp
 L Interface_USB:CP2102N-A01-GQFN28 U6
@@
 	10400 2100 10400 2050
 Wire Wire Line
-	10400 2300 10400 2350
-Wire Wire Line
 	4650 1750 4300 1750
 Wire Wire Line
@@
 GPIO39
 Wire Wire Line
-	7700 5900 8100 5900
-Wire Wire Line
-	7700 6000 8100 6000
-Wire Wire Line
-	7700 6100 8100 6100
-Wire Wire Line
-	7700 6200 8100 6200
-Wire Wire Line
-	7700 6300 8100 6300
-Text Label 7850 6200 0    50   ~ 0
+	9460 5710 9860 5710
+Wire Wire Line
+	9460 5810 9860 5810
+Wire Wire Line
+	9460 5910 9860 5910
+Wire Wire Line
+	9460 6010 9860 6010
+Wire Wire Line
+	9460 6110 9860 6110
+Text Label 9610 6010 0    50   ~ 0
 GPIO36
-Text Label 7850 6300 0    50   ~ 0
+Text Label 9610 6110 0    50   ~ 0
 GPIO39
-Text Label 7850 5900 0    50   ~ 0
+Text Label 9610 5710 0    50   ~ 0
 GPIO04
-Text Label 7850 6000 0    50   ~ 0
+Text Label 9610 5810 0    50   ~ 0
 GPIO34
-Text Label 7850 6100 0    50   ~ 0
+Text Label 9610 5910 0    50   ~ 0
 GPIO35
 Wire Wire Line
@@
 U 1 1 60DF5812
 P 10800 3550
-F 0 "R8" V 10900 3550 50  0000 C CNN
-F 1 "10k" V 10800 3550 50  0000 C CNN
+F 0 "R8" V 10880 3550 50  0000 C CNN
+F 1 "10k" V 10710 3550 50  0000 C CNN
 F 2 "Resistor_SMD:R_0402_1005Metric" V 10730 3550 50  0001 C CNN
 F 3 "~" H 10800 3550 50  0001 C CNN
@@
 U 1 1 60C6DDAB
 P 9850 1850
-F 0 "R7" V 9950 1850 50  0000 C CNN
-F 1 "4.7k" V 9850 1850 50  0000 C CNN
+F 0 "R7" V 9760 1850 50  0000 C CNN
+F 1 "4.7k" V 9940 1850 50  0000 C CNN
 F 2 "Resistor_SMD:R_0402_1005Metric" V 9780 1850 50  0001 C CNN
 F 3 "~" H 9850 1850 50  0001 C CNN
@@
 Text Notes 550  3650 0    98   ~ 20
 C64 PORTS
-Text Notes 8800 5700 0    98   ~ 20
+Text Notes 10640 5750 0    98   ~ 20
 MISC
 Text Notes 500  4100 0    98   ~ 20
@@
 U 1 1 6116524C
 P 6150 5750
-F 0 "D1" H 6000 5900 50  0000 C CNN
-F 1 "LED POWER" H 6000 5800 50  0000 C CNN
+F 0 "D1" H 5900 5840 50  0000 C CNN
+F 1 "LED POWER" H 6210 5840 50  0000 C CNN
 F 2 "LED_SMD:LED_0603_1608Metric_Pad1.05x0.95mm_HandSolder" H 6150 5750 50  0001 C CNN
 F 3 "~" H 6150 5750 50  0001 C CNN
@@
 U 1 1 61165DF4
 P 6550 5750
-F 0 "R2" V 6650 5750 50  0000 C CNN
-F 1 "150" V 6550 5750 50  0000 C CNN
+F 0 "R2" V 6620 5750 50  0000 C CNN
+F 1 "150" V 6460 5750 50  0000 C CNN
 F 2 "Resistor_SMD:R_0402_1005Metric" V 6480 5750 50  0001 C CNN
 F 3 "~" H 6550 5750 50  0001 C CNN
@@
 NoConn ~ 4650 3150
 NoConn ~ 4650 3250
-NoConn ~ 7700 5900
-NoConn ~ 7700 6000
-NoConn ~ 7700 6100
-NoConn ~ 7700 6200
-NoConn ~ 7700 6300
-$Comp
-L Mechanical:MountingHole_Pad H1
-U 1 1 60D3FB9A
-P 9100 5900
-F 0 "H1" H 9200 5949 50  0000 L CNN
-F 1 "MountingHole_Pad" H 9200 5858 50  0000 L CNN
-F 2 "MountingHole:MountingHole_3.2mm_M3_Pad" H 9100 5900 50  0001 C CNN
-F 3 "~" H 9100 5900 50  0001 C CNN
-	1    9100 5900
-	1    0    0    -1
-$EndComp
-$Comp
-L Mechanical:MountingHole_Pad H2
-U 1 1 60D4032A
-P 9350 5900
-F 0 "H2" H 9450 5949 50  0000 L CNN
-F 1 "MountingHole_Pad" H 9450 5858 50  0000 L CNN
-F 2 "MountingHole:MountingHole_3.2mm_M3_Pad" H 9350 5900 50  0001 C CNN
-F 3 "~" H 9350 5900 50  0001 C CNN
-	1    9350 5900
-	1    0    0    -1
-$EndComp
+NoConn ~ 9460 5710
+NoConn ~ 9460 5810
+NoConn ~ 9460 5910
+NoConn ~ 9460 6010
+NoConn ~ 9460 6110
 $Comp
 L Mechanical:MountingHole_Pad H3
 U 1 1 60D40B18
-P 9600 5900
-F 0 "H3" H 9700 5949 50  0000 L CNN
-F 1 "MountingHole_Pad" H 9700 5858 50  0000 L CNN
-F 2 "MountingHole:MountingHole_3.2mm_M3_Pad" H 9600 5900 50  0001 C CNN
-F 3 "~" H 9600 5900 50  0001 C CNN
-	1    9600 5900
+P 8350 5990
+F 0 "H3" H 8300 6160 50  0000 L CNN
+F 1 "MountingHole_Pad" H 8010 5810 50  0001 L CNN
+F 2 "MountingHole:MountingHole_3.2mm_M3_Pad" H 8350 5990 50  0001 C CNN
+F 3 "~" H 8350 5990 50  0001 C CNN
+	1    8350 5990
 	1    0    0    -1
 $EndComp
@@
 L Mechanical:MountingHole_Pad H4
 U 1 1 60D4139A
-P 9850 5900
-F 0 "H4" H 9950 5949 50  0000 L CNN
-F 1 "MountingHole_Pad" H 9950 5858 50  0000 L CNN
-F 2 "MountingHole:MountingHole_3.2mm_M3_Pad" H 9850 5900 50  0001 C CNN
-F 3 "~" H 9850 5900 50  0001 C CNN
-	1    9850 5900
-	1    0    0    -1
-$EndComp
-Connection ~ 10400 2300
+P 8600 5990
+F 0 "H4" H 8550 6160 50  0000 L CNN
+F 1 "MountingHole_Pad" H 8250 5810 50  0001 L CNN
+F 2 "MountingHole:MountingHole_3.2mm_M3_Pad" H 8600 5990 50  0001 C CNN
+F 3 "~" H 8600 5990 50  0001 C CNN
+	1    8600 5990
+	1    0    0    -1
+$EndComp
 $Comp
 L power:VBUS #PWR0101
@@
 Wire Wire Line
 	9550 1850 9700 1850
-NoConn ~ 9100 6000
-NoConn ~ 9350 6000
-NoConn ~ 9600 6000
-NoConn ~ 9850 6000
+NoConn ~ 7850 6090
+NoConn ~ 8100 6090
+NoConn ~ 8350 6090
+NoConn ~ 8600 6090
 $Comp
 L Graphic:Logo_Open_Hardware_Small #LOGO1
@@
 U 1 1 5F98F579
 P 6550 6000
-F 0 "R3" V 6650 6000 50  0000 C CNN
-F 1 "150" V 6550 6000 50  0000 C CNN
+F 0 "R3" V 6620 6000 50  0000 C CNN
+F 1 "150" V 6460 6000 50  0000 C CNN
 F 2 "Resistor_SMD:R_0402_1005Metric" V 6480 6000 50  0001 C CNN
 F 3 "~" H 6550 6000 50  0001 C CNN
@@
 P 4010 2310
 F 0 "R9" V 3920 2310 50  0000 C CNN
-F 1 "0" V 4010 2310 50  0000 C CNN
+F 1 "0" V 4090 2310 50  0000 C CNN
 F 2 "Resistor_SMD:R_1206_3216Metric_Pad1.30x1.75mm_HandSolder" V 3940 2310 50  0001 C CNN
 F 3 "~" H 4010 2310 50  0001 C CNN
@@
 U 1 1 5F862A7E
 P 4100 1270
-F 0 "R1" V 4000 1220 50  0000 L CNN
-F 1 "10k" V 4100 1220 50  0000 L CNN
+F 0 "R1" H 3940 1210 50  0000 L CNN
+F 1 "10k" H 3920 1290 50  0000 L CNN
 F 2 "Resistor_SMD:R_0402_1005Metric" V 4030 1270 50  0001 C CNN
 F 3 "~" H 4100 1270 50  0001 C CNN
@@
 Text Notes 9350 5380 0    50   ~ 0
 Only 2102.\nRequires additional resistors for cp2102N
+Text Notes 9120 6310 0    50   ~ 0
+Available GPIOs for future use.\nGPIOs 34-39 are Input only
+$Comp
+L Mechanical:MountingHole_Pad H1
+U 1 1 60D3FB9A
+P 7850 5990
+F 0 "H1" H 7800 6160 50  0000 L CNN
+F 1 "MountingHole_Pad" H 7510 5800 50  0001 L CNN
+F 2 "MountingHole:MountingHole_3.2mm_M3_Pad" H 7850 5990 50  0001 C CNN
+F 3 "~" H 7850 5990 50  0001 C CNN
+	1    7850 5990
+	1    0    0    -1
+$EndComp
+$Comp
+L Mechanical:MountingHole_Pad H2
+U 1 1 60D4032A
+P 8100 5990
+F 0 "H2" H 8050 6160 50  0000 L CNN
+F 1 "MountingHole_Pad" H 7760 5800 50  0001 L CNN
+F 2 "MountingHole:MountingHole_3.2mm_M3_Pad" H 8100 5990 50  0001 C CNN
+F 3 "~" H 8100 5990 50  0001 C CNN
+	1    8100 5990
+	1    0    0    -1
+$EndComp
+Wire Wire Line
+	4100 1550 3550 1550
 $EndSCHEMATC

Commit message: Unijoysticle2+ - Rev B: WIP
* 4 layer board
* hand-solder friendly
* Uses CH340C instead of CP2102
* Fixes placement of USB micro connector
Parts:
- removed C12: .1uF, Capacitor_SMD:C_0402_1005Metric, symbol Device:C_Small
- removed R7: 4.7k, Resistor_SMD:R_0402_1005Metric, symbol Device:R
- removed R8: 10k, Resistor_SMD:R_0402_1005Metric, symbol Device:R
- removed U6: CP2102, Package_DFN_QFN:QFN-28-1EP_5x5mm_P0.5mm_EP3.35x3.35mm, symbol Interface_USB:CP2102N-A01-GQFN28
- added R7, R8: 1K, Resistor_SMD:R_0805_2012Metric_Pad1.20x1.40mm_HandSolder, symbol Device:R_Small
- added U6: CH340C, Package_SO:SOIC-16_3.9x9.9mm_P1.27mm, symbol Interface_USB:CH340C
- C1, C2, C3, C4, C5, C6: footprint Capacitor_SMD:C_0402_1005Metric -> Capacitor_SMD:C_0805_2012Metric_Pad1.18x1.45mm_HandSolder
- C10: value 1uF -> .1uF; footprint Capacitor_SMD:C_0402_1005Metric -> Capacitor_SMD:C_0805_2012Metric_Pad1.18x1.45mm_HandSolder; LCSC C52923 -> (none)
- C11: footprint Capacitor_SMD:C_0402_1005Metric -> Capacitor_SMD:C_0805_2012Metric_Pad1.18x1.45mm_HandSolder; LCSC C1525 -> (none)
- C12: renamed from C13; footprint Capacitor_SMD:C_0402_1005Metric -> Capacitor_SMD:C_0805_2012Metric_Pad1.18x1.45mm_HandSolder
- C8, C9: footprint Capacitor_SMD:C_0603_1608Metric -> Capacitor_SMD:C_0805_2012Metric_Pad1.18x1.45mm_HandSolder
- D1: footprint LED_SMD:LED_0603_1608Metric_Pad1.05x0.95mm_HandSolder -> LED_SMD:LED_0805_2012Metric_Pad1.15x1.40mm_HandSolder; LCSC C72041 -> (none)
- D2: footprint LED_SMD:LED_0603_1608Metric_Pad1.05x0.95mm_HandSolder -> LED_SMD:LED_0805_2012Metric_Pad1.15x1.40mm_HandSolder; LCSC C72043 -> (none)
- D3: footprint LED_SMD:LED_0603_1608Metric_Pad1.05x0.95mm_HandSolder -> LED_SMD:LED_0805_2012Metric_Pad1.15x1.40mm_HandSolder; LCSC C72044 -> (none)
- H1, H2, H3, H4: footprint MountingHole:MountingHole_3.2mm_M3_Pad -> MountingHole:MountingHole_3.2mm_M3_Pad_Via
- R1, R5, R6: footprint Resistor_SMD:R_0402_1005Metric -> Resistor_SMD:R_0805_2012Metric_Pad1.20x1.40mm_HandSolder
- R2, R3, R4: value 150 -> 330; footprint Resistor_SMD:R_0402_1005Metric -> Resistor_SMD:R_0805_2012Metric_Pad1.20x1.40mm_HandSolder; LCSC C25082 -> (none)
Connections:
- wire segments 201 -> 196
- no-connect marks 32 -> 17
Other:
- note removed: "Only 2102.\nRequires additional resistors for cp2102N"
- moved on the sheet: D6, H1, H2, H3, H4, J3
