File: board/unijoysticle2_a500/unijoysticle2_a500.kicad_sch (KiCad schematic)
At the start: 0 parts

Commit message: Uni2 A500: Change company name
from Retro Moe to Ricardo Quesada
Other:
- company: Retro Moe -> Ricardo Quesada
Changed lines of the file:
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@@
     (date "2022-05-15")
     (rev "B")
-    (company "Retro Moe")
+    (company "Ricardo Quesada")
   )
   (sheet (at 62.23 62.23) (size 40.64 22.86) (fields_autoplaced)
