File: board/unijoysticle2_flashparty2022/unijoysticle2_flashparty.kicad_sch (KiCad schematic)
At the start: 20 parts, among them J1 DB9_Female, J2 DB9_Female, SW1 SW_Push, U1 74HC05, U2 74HC05, U3 mini_esp32

Commit message: flashparty / c64: remove warnings introduced in kicad 6.0.10
Parts:
- D3: footprint Diode_THT:D_DO-41_SOD81_P7.62mm_Horizontal -> Diode_THT:D_DO-41_SOD81_P10.16mm_Horizontal
Changed lines of the file:
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@@
       (effects (font (size 1.27 1.27)) hide)
     )
-    (property "Datasheet" "" (id 3) (at 185.42 43.18 0)
+    (property "Datasheet" " ~" (id 3) (at 185.42 43.18 0)
       (effects (font (size 1.27 1.27)) hide)
     )
@@
       (effects (font (size 1.27 1.27)) hide)
     )
-    (property "Datasheet" "" (id 3) (at 215.9 44.45 0)
+    (property "Datasheet" " ~" (id 3) (at 215.9 44.45 0)
       (effects (font (size 1.27 1.27)) hide)
     )
@@
       (effects (font (size 1.27 1.27)) hide)
     )
-    (property "Datasheet" "" (id 3) (at 29.21 185.42 0)
+    (property "Datasheet" "~" (id 3) (at 29.21 185.42 0)
       (effects (font (size 1.27 1.27)) hide)
     )
@@
     (property "Reference" "D3" (id 0) (at 154.94 183.3118 0))
     (property "Value" "1N5819" (id 1) (at 154.94 181.0004 0))
-    (property "Footprint" "Diode_THT:D_DO-41_SOD81_P7.62mm_Horizontal" (id 2) (at 154.94 173.355 0)
+    (property "Footprint" "Diode_THT:D_DO-41_SOD81_P10.16mm_Horizontal" (id 2) (at 154.94 173.355 0)
       (effects (font (size 1.27 1.27)) hide)
     )
@@
     )
     (path "/00000000-0000-0000-0000-00005f695dda"
-      (reference "D3") (unit 1) (value "1N5819") (footprint "Diode_THT:D_DO-41_SOD81_P7.62mm_Horizontal")
+      (reference "D3") (unit 1) (value "1N5819") (footprint "Diode_THT:D_DO-41_SOD81_P10.16mm_Horizontal")
     )
     (path "/00000000-0000-0000-0000-00005c705949"
