File: board/unijoysticle2_xl800/unijoysticle2_xl800.kicad_sch (KiCad schematic)
At the start: 0 parts

Commit message: 800xl: routes added
Other:
- title: Unijoysticle 2 A500 -> Unijoysticle 2 XL800
Changed lines of the file:
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@@
   (paper "A4")
   (title_block
-    (title "Unijoysticle 2 A500")
-    (date "2022-05-15")
-    (rev "B")
+    (title "Unijoysticle 2 XL800")
+    (date "2023-06-16")
+    (rev "A")
     (company "Ricardo Quesada")
   )

Commit message: Unijoysticle2 800X/A1000: fix warnings
Other:
- title: Unijoysticle 2 XL800 -> Unijoysticle 2 800XL / A1000
Changed lines of the file:
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@@
   (paper "A4")
   (title_block
-    (title "Unijoysticle 2 XL800")
-    (date "2023-06-16")
+    (title "Unijoysticle 2 800XL / A1000")
+    (date "2023-06-18")
     (rev "A")
     (company "Ricardo Quesada")
