File: board/unijoysticle2_xl800/unijoysticle2_xl800.kicad_pcb (KiCad board)
At the start: 4 copper layers, 72 x 53 mm, 58 parts, among them J1 USB_B_Micro, J2 DE9_Receptacle, J3 DE9_Receptacle, Q1 S8050, Q2 S8050, SW1 RESET, SW2 BOOT, SW3 MODE, SW4 SWAP, U1 ESP32-WROOM-32, U2 AMS1117-3.3, U3 CH340C, U4 74HC05, U5 74HC05, U6 74HC05

Commit message: show new logo
Parts:
- removed the G*** at (113.3, 110.6)
- added G***: LOGO, Unijoysticle:unijoysticle_logo_small_bis, B.Cu at (113.6, 108.2)
