File: board/unijoysticle2_c64_pico/c64_ports.kicad_sch (KiCad schematic)
At the start: 26 parts, among them J2 PORT JOY #1, J3 PORT JOY #2, SW3 MODE, SW4 SWAP, U4 74HCT05, U5 74HCT05, U6 74HCT05

Commit message: improved pico sid interrupt generation
Parts:
- R13, R14, R16, R17: value 5K1 -> 10K
- R19, R22: value 6K8 -> 10K
Other:
- note added: "10k POTX/POTY Pull-Ups (1351 Mouse & 1311/1312 Paddles)"
- note added: "10k series + 22k pull-down divides C64 POTY to 2.62V HIGH and <=0.45V LOW during SID discharge (540mV V_IL margin)."
- note added: "5V-SAFE SID SYNC DIVIDERS (10k / 22k -> 2.62V HIGH / 0.45V LOW)"
- note removed: "5.1k POTX/POTY Pull-Ups (1351 Mouse & 1311/1312 Paddles)"
- note removed: "5V-SAFE SID SYNC DIVIDERS (6.8k / 22k -> 3.24V MAX)"
- note removed: "6.8k series + 22k pull-down divides C64 5V POTY to 3.24V max (<3.6V absolute max), zero ESD diode injection."
Changed lines of the file:
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@@
 		)
 	)
-	(text "5V-SAFE SID SYNC DIVIDERS (6.8k / 22k -> 3.24V MAX)"
+	(text "5V-SAFE SID SYNC DIVIDERS (10k / 22k -> 2.62V HIGH / 0.45V LOW)"
 		(exclude_from_sim no)
 		(at 130.81 126.746 0)
@@
 		)
 	)
-	(text "6.8k series + 22k pull-down divides C64 5V POTY\nto 3.24V max (<3.6V absolute max), zero ESD diode injection."
+	(text "10k series + 22k pull-down divides C64 POTY to 2.62V HIGH\nand <=0.45V LOW during SID discharge (540mV V_IL margin)."
 		(exclude_from_sim no)
 		(at 130.81 134.62 0)
@@
 		)
 	)
-	(text "5.1k POTX/POTY Pull-Ups (1351 Mouse & 1311/1312 Paddles)"
+	(text "10k POTX/POTY Pull-Ups (1351 Mouse & 1311/1312 Paddles)"
 		(exclude_from_sim no)
 		(at 35.433 104.648 0)
@@
 			)
 		)
-		(property "Value" "5K1"
+		(property "Value" "10K"
 			(at 38.1 97.0279 0)
 			(show_name no)
@@
 			)
 		)
-		(property "Value" "5K1"
+		(property "Value" "10K"
 			(at 73.66 97.0279 0)
 			(show_name no)
@@
 			)
 		)
-		(property "Value" "6K8"
+		(property "Value" "10K"
 			(at 151.13 165.735 90)
 			(show_name no)
@@
 			)
 		)
-		(property "Value" "6K8"
+		(property "Value" "10K"
 			(at 151.13 145.415 90)
 			(show_name no)
@@
 			)
 		)
-		(property "Value" "5K1"
+		(property "Value" "10K"
 			(at 62.23 97.0279 0)
 			(show_name no)
@@
 			)
 		)
-		(property "Value" "5K1"
+		(property "Value" "10K"
 			(at 49.53 97.0279 0)
 			(show_name no)

Commit message: Unijoysticle C64 Pico board
Parts:
- J2, J3: footprint Connector_Dsub:DSUB-9_Female_Horizontal_P2.77x2.54mm_EdgePinOffset9.40mm -> Connector_Dsub:DSUB-9_Socket_Horizontal_P2.77x2.54mm_EdgePinOffset9.40mm
Changed lines of the file:
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@@
 			)
 		)
-		(property "Footprint" "Connector_Dsub:DSUB-9_Female_Horizontal_P2.77x2.54mm_EdgePinOffset9.40mm"
+		(property "Footprint" "Connector_Dsub:DSUB-9_Socket_Horizontal_P2.77x2.54mm_EdgePinOffset9.40mm"
 			(at 45.212 47.752 0)
 			(hide yes)
@@
 			)
 		)
-		(property "Footprint" "Connector_Dsub:DSUB-9_Female_Horizontal_P2.77x2.54mm_EdgePinOffset9.40mm"
+		(property "Footprint" "Connector_Dsub:DSUB-9_Socket_Horizontal_P2.77x2.54mm_EdgePinOffset9.40mm"
 			(at 62.992 47.752 0)
 			(hide yes)

Commit message: JLCPCB parts
Parts:
- C11, C12, C13: LCSC (none) -> C49678; MPN (none) -> CC0805KRX7R9BB104; Manufacturer (none) -> YAGEO
- D4: LCSC (none) -> C84259; MPN (none) -> NCD0805B2; Manufacturer (none) -> Foshan NationStar Optoelectronics
- D5: LCSC (none) -> C2297; MPN (none) -> KT-0805G; Manufacturer (none) -> Hubei KENTO Elec
- D6: LCSC (none) -> C84256; MPN (none) -> NCD0805R1; Manufacturer (none) -> Foshan NationStar Optoelectronics
- R10, R11, R13, R14, R16, R17, R19, R22: LCSC (none) -> C17414; MPN (none) -> 0805W8F1002T5E; Manufacturer (none) -> UNI-ROYAL
- R20, R23: LCSC (none) -> C17560; MPN (none) -> 0805W8F2202T5E; Manufacturer (none) -> UNI-ROYAL
- R7, R8, R9: LCSC (none) -> C26010; MPN (none) -> 0805W8F3301T5E; Manufacturer (none) -> UNI-ROYAL
- SW3, SW4: MPN (none) -> PTS645VH39-2 LFS; Manufacturer (none) -> C&K
- U4, U5, U6: LCSC (none) -> C49188197; MPN (none) -> EM74HCT05D; Manufacturer (none) -> EnergyMath
