File: board/unijoysticle2_c64_pico/pico2w.kicad_sch (KiCad schematic)
At the start: 11 parts, among them J4 DEBUG_LA_HDR, SW1 RESET, U1 Raspberry_Pi_Pico_2_W

Commit message: Unijoysticle C64 Pico board
Parts:
- U1: footprint MCU_RaspberryPi_and_Boards:RPi_Pico_SMD_TH -> Unijoysticle:RPi_Pico_2_W_SMD_TH
Changed lines of the file:
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@@
 			)
 		)
-		(property "Footprint" "MCU_RaspberryPi_and_Boards:RPi_Pico_SMD_TH"
+		(property "Footprint" "Unijoysticle:RPi_Pico_2_W_SMD_TH"
 			(at 114.3 88.9 90)
 			(hide yes)

Commit message: JLCPCB parts
Parts:
- C1, C4: LCSC (none) -> C49678; MPN (none) -> CC0805KRX7R9BB104; Manufacturer (none) -> YAGEO
- C5: LCSC (none) -> C15850; MPN (none) -> CL21A106KAYNNNE; Manufacturer (none) -> Samsung Electro-Mechanics
- D1: LCSC (none) -> C2297; MPN (none) -> KT-0805G; Manufacturer (none) -> Hubei KENTO Elec
- R1: LCSC (none) -> C17414; MPN (none) -> 0805W8F1002T5E; Manufacturer (none) -> UNI-ROYAL
- R2: LCSC (none) -> C26010; MPN (none) -> 0805W8F3301T5E; Manufacturer (none) -> UNI-ROYAL
- SW1: MPN (none) -> PTS645VH39-2 LFS; Manufacturer (none) -> C&K
- U1: MPN (none) -> SC1633; Manufacturer (none) -> Raspberry Pi
