File: board/unijoysticle2_c64_pico/power.kicad_sch (KiCad schematic)
At the start: 10 parts, among them Q1 DMG2305UX

Commit message: removed unneeded diode in power filtering
Parts:
- removed D2: 1N5819, Diode_SMD:D_SOD-123, symbol Device:D_Schottky_Small
Other:
- note added: "ZERO-DROP P-FET IDEAL DIODE + USB VBUS OR-ING (Pico 2 W Datasheet Section 3.5, Figure 10, pp. 15-16) - When USB is unplugged (VBUS=0V): R3 (+ Pico internal 20k) pulls Q1 Gate to GND, turning Q1 fully ON (Rds_on = 52mOhm, <3mV drop at 45mA). - When USB is plugged in (VBUS=5V): Q1 Gate is pulled to 5V, turning Q1 OFF to block back-feeding into C64 +5V while Pico onboard D1 powers VSYS."
- note removed: "ZERO-DROP P-FET IDEAL DIODE + USB VBUS OR-ING (Pico 2 W Datasheet Section 3.4, Figure 10, p. 16) - When USB is unplugged (VBUS=0V): R3 pulls Q1 Gate to GND, turning Q1 fully ON (Rds_on = 52mOhm, <3mV drop at 45mA). - When USB is plugged in (VBUS=5V): Q1 Gate is pulled to 5V, turning Q1 OFF to block back-feeding into C64 +5V rail."
Changed lines of the file:
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@@
 		)
 	)
-	(text "ZERO-DROP P-FET IDEAL DIODE + USB VBUS OR-ING\n(Pico 2 W Datasheet Section 3.4, Figure 10, p. 16)\n- When USB is unplugged (VBUS=0V): R3 pulls Q1 Gate to GND,\n  turning Q1 fully ON (Rds_on = 52mOhm, <3mV drop at 45mA).\n- When USB is plugged in (VBUS=5V): Q1 Gate is pulled to 5V,\n  turning Q1 OFF to block back-feeding into C64 +5V rail."
+	(text "ZERO-DROP P-FET IDEAL DIODE + USB VBUS OR-ING\n(Pico 2 W Datasheet Section 3.5, Figure 10, pp. 15-16)\n- When USB is unplugged (VBUS=0V): R3 (+ Pico internal 20k) pulls Q1 Gate to GND,\n  turning Q1 fully ON (Rds_on = 52mOhm, <3mV drop at 45mA).\n- When USB is plugged in (VBUS=5V): Q1 Gate is pulled to 5V, turning Q1 OFF\n  to block back-feeding into C64 +5V while Pico onboard D1 powers VSYS."
 		(exclude_from_sim no)
 		(at 35.56 114.3 0)
@@
 	)
 	(junction
-		(at 109.22 71.12)
-		(diameter 0)
-		(color 0 0 0 0)
-	)
-	(junction
 		(at 119.38 71.12)
 		(diameter 0)
@@
 	(wire
 		(pts
-			(xy 91.44 81.28) (xy 96.52 81.28)
-		)
-		(stroke
-			(width 0)
-			(type default)
-		)
-	)
-	(wire
-		(pts
-			(xy 101.6 81.28) (xy 109.22 81.28)
-		)
-		(stroke
-			(width 0)
-			(type default)
-		)
-	)
-	(wire
-		(pts
-			(xy 109.22 81.28) (xy 109.22 71.12)
-		)
-		(stroke
-			(width 0)
-			(type default)
-		)
-	)
-	(wire
-		(pts
 			(xy 99.06 66.04) (xy 99.06 71.12)
 		)
@@
 	(wire
 		(pts
-			(xy 99.06 71.12) (xy 109.22 71.12)
-		)
-		(stroke
-			(width 0)
-			(type default)
-		)
-	)
-	(wire
-		(pts
-			(xy 109.22 71.12) (xy 119.38 71.12)
+			(xy 99.06 71.12) (xy 119.38 71.12)
 		)
 		(stroke
@@
 					(unit 1)
 				)
-			)
-		)
-	)
-	(symbol
-		(lib_id "Device:D_Schottky_Small")
-		(at 99.06 81.28 180)
-		(unit 1)
-		(body_style 1)
-		(exclude_from_sim no)
-		(in_bom yes)
-		(on_board yes)
-		(in_pos_files yes)
-		(dnp no)
-		(property "Reference" "D2"
-			(at 99.06 77.47 0)
-			(show_name no)
-			(do_not_autoplace no)
-			(effects
-				(font
-					(size 1.27 1.27)
-				)
-			)
-		)
-		(property "Value" "1N5819"
-			(at 99.06 85.09 0)
-			(show_name no)
-			(do_not_autoplace no)
-			(effects
-				(font
-					(size 1.27 1.27)
-				)
-			)
-		)
-		(property "Footprint" "Diode_SMD:D_SOD-123"
-			(at 99.06 81.28 90)
-			(hide yes)
-			(show_name no)
-			(do_not_autoplace no)
-			(effects
-				(font
-					(size 1.27 1.27)
-				)
-			)
-		)
-		(property "Datasheet" ""
-			(at 99.06 81.28 90)
-			(hide yes)
-			(show_name no)
-			(do_not_autoplace no)
-			(effects
-				(font
-					(size 1.27 1.27)
-				)
-			)
-		)
-		(property "Description" ""
-			(at 99.06 81.28 0)
-			(show_name no)
-			(do_not_autoplace no)
-			(effects
-				(font
-					(size 1.27 1.27)
-				)
-			)
-		)
-		(pin "1"
-		)
-		(pin "2"
-		)
-		(instances
-			(project "unijoysticle2_c64_pico"
-				(path "/0e6b6c40-efab-4794-bc88-ed2592ffa1bd/93281dcd-2548-47fa-896a-a960429efc33"
-					(reference "D2")
-					(unit 1)
-				)

Commit message: JLCPCB parts
Parts:
- C10, C8: LCSC (none) -> C49678; MPN (none) -> CC0805KRX7R9BB104; Manufacturer (none) -> YAGEO
- C6, C9: LCSC (none) -> C15850; MPN (none) -> CL21A106KAYNNNE; Manufacturer (none) -> Samsung Electro-Mechanics
- C7: LCSC (none) -> C124129; MPN (none) -> GRM21BR61A476ME15L; Manufacturer (none) -> Murata Electronics
- F1: LCSC (none) -> C20608679; MPN (none) -> 0805L025/36XR; Manufacturer (none) -> LUTE
- FB1: LCSC (none) -> C1017; MPN (none) -> GZ2012D601TF; Manufacturer (none) -> Sunlord
- Q1: LCSC (none) -> C144153; MPN (none) -> DMG2305UX-13; Manufacturer (none) -> Diodes Incorporated
- R3: LCSC (none) -> C149504; MPN (none) -> 0805W8F1003T5E; Manufacturer (none) -> UNI-ROYAL
