File: board/unijoysticle2_c64_pico/unijoysticle2_c64_pico.kicad_pcb (KiCad board)
At the start: 4 copper layers, 62.5 x 60 mm, 48 parts, among them J2 PORT JOY #1, J3 PORT JOY #2, J4 DEBUG_LA_HDR, Q1 DMG2305UX, SW1 RESET, SW3 MODE, SW4 SWAP, U1 Raspberry_Pi_Pico_2_W, U4 74HCT05, U5 74HCT05, U6 74HCT05

Commit message: pico license
Parts:
- LOGO1: value OSHW -> CC_BY-NC-SA_4.0; footprint OSHW-Symbol_6.7x6mm_SilkScreen -> Unijoysticle:CC_BY_NC_SA_4_0_SilkScreen
- moved LOGO1 3.24 mm to (129.3, 115.3)
Other:
- board text added: "retro.moe - CC BY-NC-SA 4.0"
- board text removed: "retro.moe - Open Hardware"
