File: board/unipad_c64/c64_ports.kicad_sch (KiCad schematic)
At the start: 26 parts, among them J2 PORT JOY #1, J3 PORT JOY #2, SW3 MODE, SW4 SWAP, U4 74HCT05, U5 74HCT05, U6 74HCT05

Commit message: unipad c64
Other:
- title: Unijoysticle 2 C64 (DB9 Ports, 74HCT05 & SID SYNC) -> Unipad C64 (Control Ports, 74HCT05 & SID SYNC)
