File: board/unipad_c64/pico2w.kicad_sch (KiCad schematic)
At the start: 11 parts, among them J4 DEBUG_LA_HDR, SW1 RESET, U1 Raspberry_Pi_Pico_2_W

Commit message: unipad c64
Other:
- title: Unijoysticle 2 C64 (Pico 2 W & Debug) -> Unipad C64 (MCU & Debug)
Changed lines of the file:
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@@
 	(paper "A4")
 	(title_block
-		(title "Unijoysticle 2 C64 (Pico 2 W & Debug)")
+		(title "Unipad C64 (MCU & Debug)")
 		(date "2026-10-26")
-		(rev "D")
+		(rev "A")
 		(company "Ricardo Quesada")
 		(comment 1 "Raspberry Pi Pico 2 W (RP2350 + CYW43439) + 1x8 Debug Header")
@@
 		)
 		(instances
-			(project "unijoysticle2_c64_pico"
+			(project "unipad_c64"
 				(path "/0e6b6c40-efab-4794-bc88-ed2592ffa1bd/4c2fb79c-207e-4f92-8ea1-7543e9ed400d"
 					(reference "U1")
@@
 		)
 		(instances
-			(project "unijoysticle2_c64_pico"
+			(project "unipad_c64"
 				(path "/0e6b6c40-efab-4794-bc88-ed2592ffa1bd/4c2fb79c-207e-4f92-8ea1-7543e9ed400d"
 					(reference "J4")
@@
 		)
 		(instances
-			(project "unijoysticle2_c64_pico"
+			(project "unipad_c64"
 				(path "/0e6b6c40-efab-4794-bc88-ed2592ffa1bd/4c2fb79c-207e-4f92-8ea1-7543e9ed400d"
 					(reference "SW1")
@@
 		)
 		(instances
-			(project "unijoysticle2_c64_pico"
+			(project "unipad_c64"
 				(path "/0e6b6c40-efab-4794-bc88-ed2592ffa1bd/4c2fb79c-207e-4f92-8ea1-7543e9ed400d"
 					(reference "C1")
@@
 		)
 		(instances
-			(project "unijoysticle2_c64_pico"
+			(project "unipad_c64"
 				(path "/0e6b6c40-efab-4794-bc88-ed2592ffa1bd/4c2fb79c-207e-4f92-8ea1-7543e9ed400d"
 					(reference "R1")
@@
 		)
 		(instances
-			(project "unijoysticle2_c64_pico"
+			(project "unipad_c64"
 				(path "/0e6b6c40-efab-4794-bc88-ed2592ffa1bd/4c2fb79c-207e-4f92-8ea1-7543e9ed400d"
 					(reference "C4")
@@
 		)
 		(instances
-			(project "unijoysticle2_c64_pico"
+			(project "unipad_c64"
 				(path "/0e6b6c40-efab-4794-bc88-ed2592ffa1bd/4c2fb79c-207e-4f92-8ea1-7543e9ed400d"
 					(reference "C5")
@@
 		)
 		(instances
-			(project "unijoysticle2_c64_pico"
+			(project "unipad_c64"
 				(path "/0e6b6c40-efab-4794-bc88-ed2592ffa1bd/4c2fb79c-207e-4f92-8ea1-7543e9ed400d"
 					(reference "D1")
@@
 		)
 		(instances
-			(project "unijoysticle2_c64_pico"
+			(project "unipad_c64"
 				(path "/0e6b6c40-efab-4794-bc88-ed2592ffa1bd/4c2fb79c-207e-4f92-8ea1-7543e9ed400d"
 					(reference "R2")
@@
 		)
 		(instances
-			(project "unijoysticle2_c64_pico"
+			(project "unipad_c64"
 				(path "/0e6b6c40-efab-4794-bc88-ed2592ffa1bd/4c2fb79c-207e-4f92-8ea1-7543e9ed400d"
 					(reference "H1")
@@
 		)
 		(instances
-			(project "unijoysticle2_c64_pico"
+			(project "unipad_c64"
 				(path "/0e6b6c40-efab-4794-bc88-ed2592ffa1bd/4c2fb79c-207e-4f92-8ea1-7543e9ed400d"
 					(reference "H2")
@@
 		)
 		(instances
-			(project "unijoysticle2_c64_pico"
+			(project "unipad_c64"
 				(path "/0e6b6c40-efab-4794-bc88-ed2592ffa1bd/4c2fb79c-207e-4f92-8ea1-7543e9ed400d"
 					(reference "#PWR01")
@@
 		)
 		(instances
-			(project "unijoysticle2_c64_pico"
+			(project "unipad_c64"
 				(path "/0e6b6c40-efab-4794-bc88-ed2592ffa1bd/4c2fb79c-207e-4f92-8ea1-7543e9ed400d"
 					(reference "#PWR02")
@@
 		)
 		(instances
-			(project "unijoysticle2_c64_pico"
+			(project "unipad_c64"
 				(path "/0e6b6c40-efab-4794-bc88-ed2592ffa1bd/4c2fb79c-207e-4f92-8ea1-7543e9ed400d"
 					(reference "#PWR03")
@@
 		)
 		(instances
-			(project "unijoysticle2_c64_pico"
+			(project "unipad_c64"
 				(path "/0e6b6c40-efab-4794-bc88-ed2592ffa1bd/4c2fb79c-207e-4f92-8ea1-7543e9ed400d"
 					(reference "#PWR04")
@@
 		)
 		(instances
-			(project "unijoysticle2_c64_pico"
+			(project "unipad_c64"
 				(path "/0e6b6c40-efab-4794-bc88-ed2592ffa1bd/4c2fb79c-207e-4f92-8ea1-7543e9ed400d"
 					(reference "#PWR05")
@@
 		)
 		(instances
-			(project "unijoysticle2_c64_pico"
+			(project "unipad_c64"
 				(path "/0e6b6c40-efab-4794-bc88-ed2592ffa1bd/4c2fb79c-207e-4f92-8ea1-7543e9ed400d"
 					(reference "#PWR06")
@@
 		)
 		(instances
-			(project "unijoysticle2_c64_pico"
+			(project "unipad_c64"
 				(path "/0e6b6c40-efab-4794-bc88-ed2592ffa1bd/4c2fb79c-207e-4f92-8ea1-7543e9ed400d"
 					(reference "#PWR07")
@@
 		)
 		(instances
-			(project "unijoysticle2_c64_pico"
+			(project "unipad_c64"
 				(path "/0e6b6c40-efab-4794-bc88-ed2592ffa1bd/4c2fb79c-207e-4f92-8ea1-7543e9ed400d"
 					(reference "#PWR08")
@@
 		)
 		(instances
-			(project "unijoysticle2_c64_pico"
+			(project "unipad_c64"
 				(path "/0e6b6c40-efab-4794-bc88-ed2592ffa1bd/4c2fb79c-207e-4f92-8ea1-7543e9ed400d"
 					(reference "#PWR09")
@@
 		)
 		(instances
-			(project "unijoysticle2_c64_pico"
+			(project "unipad_c64"
 				(path "/0e6b6c40-efab-4794-bc88-ed2592ffa1bd/4c2fb79c-207e-4f92-8ea1-7543e9ed400d"
 					(reference "#PWR010")
@@
 		)
 		(instances
-			(project "unijoysticle2_c64_pico"
+			(project "unipad_c64"
 				(path "/0e6b6c40-efab-4794-bc88-ed2592ffa1bd/4c2fb79c-207e-4f92-8ea1-7543e9ed400d"
 					(reference "#PWR011")
@@
 		)
 		(instances
-			(project "unijoysticle2_c64_pico"
+			(project "unipad_c64"
 				(path "/0e6b6c40-efab-4794-bc88-ed2592ffa1bd/4c2fb79c-207e-4f92-8ea1-7543e9ed400d"
 					(reference "#PWR012")
@@
 		)
 		(instances
-			(project "unijoysticle2_c64_pico"
+			(project "unipad_c64"
 				(path "/0e6b6c40-efab-4794-bc88-ed2592ffa1bd/4c2fb79c-207e-4f92-8ea1-7543e9ed400d"
 					(reference "#PWR013")
@@
 		)
 		(instances
-			(project "unijoysticle2_c64_pico"
+			(project "unipad_c64"
 				(path "/0e6b6c40-efab-4794-bc88-ed2592ffa1bd/4c2fb79c-207e-4f92-8ea1-7543e9ed400d"
 					(reference "#PWR014")
@@
 		)
 		(instances
-			(project "unijoysticle2_c64_pico"
+			(project "unipad_c64"
 				(path "/0e6b6c40-efab-4794-bc88-ed2592ffa1bd/4c2fb79c-207e-4f92-8ea1-7543e9ed400d"
 					(reference "#PWR015")
