File: board/unipad_c64/power.kicad_sch (KiCad schematic)
At the start: 9 parts, among them Q1 DMG2305UX

Commit message: unipad c64
Other:
- title: Unijoysticle 2 C64 (Power & Filtering) -> Unipad C64 (Power & Filtering)
Changed lines of the file:
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@@
 	(paper "A4")
 	(title_block
-		(title "Unijoysticle 2 C64 (Power & Filtering)")
+		(title "Unipad C64 (Power & Filtering)")
 		(date "2026-10-26")
-		(rev "D")
+		(rev "A")
 		(company "Ricardo Quesada")
 		(comment 1 "250mA PTC Polyfuse + Ferrite Pi-Filter + DMG2305UX Ideal Diode OR-ing")
@@
 		)
 		(instances
-			(project "unijoysticle2_c64_pico"
+			(project "unipad_c64"
 				(path "/0e6b6c40-efab-4794-bc88-ed2592ffa1bd/93281dcd-2548-47fa-896a-a960429efc33"
 					(reference "#PWR020")
@@
 		)
 		(instances
-			(project "unijoysticle2_c64_pico"
+			(project "unipad_c64"
 				(path "/0e6b6c40-efab-4794-bc88-ed2592ffa1bd/93281dcd-2548-47fa-896a-a960429efc33"
 					(reference "F1")
@@
 		)
 		(instances
-			(project "unijoysticle2_c64_pico"
+			(project "unipad_c64"
 				(path "/0e6b6c40-efab-4794-bc88-ed2592ffa1bd/93281dcd-2548-47fa-896a-a960429efc33"
 					(reference "C6")
@@
 		)
 		(instances
-			(project "unijoysticle2_c64_pico"
+			(project "unipad_c64"
 				(path "/0e6b6c40-efab-4794-bc88-ed2592ffa1bd/93281dcd-2548-47fa-896a-a960429efc33"
 					(reference "#PWR021")
@@
 		)
 		(instances
-			(project "unijoysticle2_c64_pico"
+			(project "unipad_c64"
 				(path "/0e6b6c40-efab-4794-bc88-ed2592ffa1bd/93281dcd-2548-47fa-896a-a960429efc33"
 					(reference "FB1")
@@
 		)
 		(instances
-			(project "unijoysticle2_c64_pico"
+			(project "unipad_c64"
 				(path "/0e6b6c40-efab-4794-bc88-ed2592ffa1bd/93281dcd-2548-47fa-896a-a960429efc33"
 					(reference "C7")
@@
 		)
 		(instances
-			(project "unijoysticle2_c64_pico"
+			(project "unipad_c64"
 				(path "/0e6b6c40-efab-4794-bc88-ed2592ffa1bd/93281dcd-2548-47fa-896a-a960429efc33"
 					(reference "#PWR022")
@@
 		)
 		(instances
-			(project "unijoysticle2_c64_pico"
+			(project "unipad_c64"
 				(path "/0e6b6c40-efab-4794-bc88-ed2592ffa1bd/93281dcd-2548-47fa-896a-a960429efc33"
 					(reference "C8")
@@
 		)
 		(instances
-			(project "unijoysticle2_c64_pico"
+			(project "unipad_c64"
 				(path "/0e6b6c40-efab-4794-bc88-ed2592ffa1bd/93281dcd-2548-47fa-896a-a960429efc33"
 					(reference "#PWR023")
@@
 		)
 		(instances
-			(project "unijoysticle2_c64_pico"
+			(project "unipad_c64"
 				(path "/0e6b6c40-efab-4794-bc88-ed2592ffa1bd/93281dcd-2548-47fa-896a-a960429efc33"
 					(reference "Q1")
@@
 		)
 		(instances
-			(project "unijoysticle2_c64_pico"
+			(project "unipad_c64"
 				(path "/0e6b6c40-efab-4794-bc88-ed2592ffa1bd/93281dcd-2548-47fa-896a-a960429efc33"
 					(reference "#PWR024")
@@
 		)
 		(instances
-			(project "unijoysticle2_c64_pico"
+			(project "unipad_c64"
 				(path "/0e6b6c40-efab-4794-bc88-ed2592ffa1bd/93281dcd-2548-47fa-896a-a960429efc33"
 					(reference "R3")
@@
 		)
 		(instances
-			(project "unijoysticle2_c64_pico"
+			(project "unipad_c64"
 				(path "/0e6b6c40-efab-4794-bc88-ed2592ffa1bd/93281dcd-2548-47fa-896a-a960429efc33"
 					(reference "#PWR025")
@@
 		)
 		(instances
-			(project "unijoysticle2_c64_pico"
+			(project "unipad_c64"
 				(path "/0e6b6c40-efab-4794-bc88-ed2592ffa1bd/93281dcd-2548-47fa-896a-a960429efc33"
 					(reference "C9")
@@
 		)
 		(instances
-			(project "unijoysticle2_c64_pico"
+			(project "unipad_c64"
 				(path "/0e6b6c40-efab-4794-bc88-ed2592ffa1bd/93281dcd-2548-47fa-896a-a960429efc33"
 					(reference "#PWR026")
@@
 		)
 		(instances
-			(project "unijoysticle2_c64_pico"
+			(project "unipad_c64"
 				(path "/0e6b6c40-efab-4794-bc88-ed2592ffa1bd/93281dcd-2548-47fa-896a-a960429efc33"
 					(reference "C10")
@@
 		)
 		(instances
-			(project "unijoysticle2_c64_pico"
+			(project "unipad_c64"
 				(path "/0e6b6c40-efab-4794-bc88-ed2592ffa1bd/93281dcd-2548-47fa-896a-a960429efc33"
 					(reference "#PWR027")
@@
 		)
 		(instances
-			(project "unijoysticle2_c64_pico"
+			(project "unipad_c64"
 				(path "/0e6b6c40-efab-4794-bc88-ed2592ffa1bd/93281dcd-2548-47fa-896a-a960429efc33"
 					(reference "#PWR028")
@@
 		)
 		(instances
-			(project "unijoysticle2_c64_pico"
+			(project "unipad_c64"
 				(path "/0e6b6c40-efab-4794-bc88-ed2592ffa1bd/93281dcd-2548-47fa-896a-a960429efc33"
 					(reference "#FLG01")
@@
 		)
 		(instances
-			(project "unijoysticle2_c64_pico"
+			(project "unipad_c64"
 				(path "/0e6b6c40-efab-4794-bc88-ed2592ffa1bd/93281dcd-2548-47fa-896a-a960429efc33"
 					(reference "#FLG02")
