File: board/unipad_c64/unipad_c64.kicad_pcb (KiCad board)
At the start: 4 copper layers, 62.5 x 60 mm, 48 parts, among them J2 PORT JOY #1, J3 PORT JOY #2, J4 DEBUG_LA_HDR, Q1 DMG2305UX, SW1 RESET, SW3 MODE, SW4 SWAP, U1 Raspberry_Pi_Pico_2_W, U4 74HCT05, U5 74HCT05, U6 74HCT05

Commit message: unipad c64
Other:
- board text added: "PORT #1"
- board text added: "PORT #2"
- board text added: "PORT1"
- board text added: "PORT2"
- board text added: "Rev. A - Gamepad · Paddle · Mouse"
- board text added: "Unipad C64"
- board text removed: "JOY1"
- board text removed: "JOY2"
- board text removed: "PORT JOY #1"
- board text removed: "PORT JOY #2"
- board text removed: "Rev. D - RP2350 + CYW43439"
- board text removed: "Unijoysticle 2 C64 Pico"
Changed lines of the file:
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@@
 	(paper "A4")
 	(title_block
-		(title "Unijoysticle 2 C64 (Pico 2 W Edition)")
+		(title "Unipad C64")
 		(date "2026-10-26")
-		(rev "D")
+		(rev "A")
 		(company "Ricardo Quesada")
-		(comment 1 "4-Layer PCB (F.Cu / In1.Cu GND / In2.Cu GND / B.Cu) - Raspberry Pi Pico 2 W")
+		(comment 1 "4-Layer PCB - Wireless Gamepad, Paddle & 1351 Mouse Adapter for Commodore 64")
 		(comment 2 "License: CC BY-NC-SA 4.0 (Attribution-NonCommercial-ShareAlike 4.0)")
 	)
@@
 		)
 	)
-	(gr_text "JOY1"
-		(at 91.7 106.24 0)
+	(gr_text "PORT1"
+		(at 92.65 106.24 0)
 		(layer "F.SilkS")
 		(effects
@@
 		)
 	)
-	(gr_text "JOY2"
-		(at 91.7 110.53 0)
+	(gr_text "PORT2"
+		(at 92.65 110.53 0)
 		(layer "F.SilkS")
 		(effects
@@
 		)
 	)
-	(gr_text "PORT JOY #1"
-		(at 94.5 97.2 0)
+	(gr_text "Unipad C64"
+		(at 110.8 93.7 0)
+		(layer "F.SilkS")
+		(effects
+			(font
+				(size 1.15 1.15)
+				(thickness 0.19)
+			)
+		)
+	)
+	(gr_text "PORT #1"
+		(at 95.8 97.45 0)
 		(layer "F.SilkS")
 		(effects
@@
 		)
 	)
-	(gr_text "PORT JOY #2"
-		(at 126 97.2 0)
+	(gr_text "PORT #2"
+		(at 127 97.45 0)
 		(layer "F.SilkS")
 		(effects
@@
 	)
 	(gr_text "(c) 2026 Ricardo Quesada"
-		(at 127 131.6 0)
+		(at 128 131.65 0)
 		(layer "B.SilkS")
 		(effects
@@
 	)
 	(gr_text "retro.moe  -  CC BY-NC-SA 4.0"
-		(at 127 133.8 0)
+		(at 128 133.85 0)
 		(layer "B.SilkS")
 		(effects
@@
 		)
 	)
-	(gr_text "Rev. D  -  RP2350 + CYW43439"
-		(at 127 129 0)
+	(gr_text "Rev. A - Gamepad · Paddle · Mouse"
+		(at 128 129.25 0)
 		(layer "B.SilkS")
 		(effects
 			(font
-				(size 0.85 0.85)
-				(thickness 0.14)
+				(size 0.8 0.8)
+				(thickness 0.13)
 			)
 			(justify mirror)
 		)
 	)
-	(gr_text "Unijoysticle 2 C64 Pico"
-		(at 127 126.2 0)
+	(gr_text "Unipad C64"
+		(at 128 126.2 0)
 		(layer "B.SilkS")
 		(effects
 			(font
-				(size 1.25 1.25)
-				(thickness 0.2)
+				(size 1.45 1.45)
+				(thickness 0.24)
 			)
 			(justify mirror)
